File: Hardware Design/GPS_board_v3.kicad_pcb (KiCad board)
At the start: 2 copper layers, 50 x 77.5 mm, 20 parts, among them IC2 SN65HVD231QDR, U1 STM32F042F4Px, U5 MAX-M8W

Commit message: final updated board + prod files
Parts:
- removed J1: ~, Connector_PinHeader_2.54mm:PinHeader_1x02_P2.54mm_Vertical
Routing:
- net SCL: track 55.5 -> 0.00 mm
- net SDA: track 55.0 -> 0.00 mm
Other:
- board text added: "CAN R (SHORT)"
